Commit message: fix?

File: picar.urdf (robot description, URDF)
Before this commit: robot picar, 5 links, 4 joints
Links:
- added link camera_link, mass 0.05; collision box size=0.04 0.06 0.04; visual box size=0.04 0.06 0.04
- link base_link: mass 1.0 -> 1.8; geometry collision box size=0.26 0.17 0.06; visual box size=0.26 0.17 0.06
- link wheel_fl: mass 0.1 -> 0.05; geometry collision cylinder length=0.03 radius=0.032; visual cylinder length=0.03 radius=0.032
- link wheel_fr: mass 0.1 -> 0.05; geometry collision cylinder length=0.03 radius=0.032; visual cylinder length=0.03 radius=0.032
- link wheel_rl: mass 0.1 -> 0.12; geometry collision cylinder length=0.04 radius=0.035; visual cylinder length=0.04 radius=0.035
- link wheel_rr: mass 0.1 -> 0.12; geometry collision cylinder length=0.04 radius=0.035; visual cylinder length=0.04 radius=0.035
Joints:
- added joint camera_joint: type fixed, parent base_link, child camera_link, origin xyz=0.14 0 0.10 rpy=0 0 0
- joint joint_fl: limit (none) -> effort=20.0 velocity=30.0; origin xyz=0.1 0.08 -0.02 -> xyz=0.13 0.085 -0.032
- joint joint_fr: limit (none) -> effort=20.0 velocity=30.0; origin xyz=0.1 -0.08 -0.02 -> xyz=0.13 -0.085 -0.032
- joint joint_rl: limit (none) -> effort=20.0 velocity=30.0; origin xyz=-0.1 0.08 -0.02 -> xyz=-0.13 0.085 -0.035
- joint joint_rr: limit (none) -> effort=20.0 velocity=30.0; origin xyz=-0.1 -0.08 -0.02 -> xyz=-0.13 -0.085 -0.035

Commit message: ehhh?

File: picar.urdf (robot description, URDF)
Before this commit: robot picar, 6 links, 5 joints
Joints:
- joint camera_joint: origin xyz=0.14 0 0.10 rpy=0 0 0 -> xyz=0.14 0 0.10 rpy=0 -0.17 0
- joint joint_fl: limit effort=20.0 velocity=30.0 -> effort=20.0 velocity=40.0
- joint joint_fr: limit effort=20.0 velocity=30.0 -> effort=20.0 velocity=40.0
- joint joint_rl: limit effort=20.0 velocity=30.0 -> effort=20.0 velocity=40.0
- joint joint_rr: limit effort=20.0 velocity=30.0 -> effort=20.0 velocity=40.0

Commit message: boogaloo

File: picar.urdf (robot description, URDF)
Before this commit: robot picar, 6 links, 5 joints
Links:
- removed link camera_link
- removed link wheel_fl
- removed link wheel_fr
- removed link wheel_rl
- removed link wheel_rr
- added link fl_steering_knuckle, mass 0.01; visual cylinder length=0.01 radius=0.005
- added link fl_wheel, mass 0.05; collision cylinder length=0.025 radius=0.0325; visual cylinder length=0.025 radius=0.0325
- added link fr_steering_knuckle, mass 0.01; visual cylinder length=0.01 radius=0.005
- added link fr_wheel, mass 0.05; collision cylinder length=0.025 radius=0.0325; visual cylinder length=0.025 radius=0.0325
- added link rl_wheel, mass 0.05; collision cylinder length=0.025 radius=0.0325; visual cylinder length=0.025 radius=0.0325
- added link rr_wheel, mass 0.05; collision cylinder length=0.025 radius=0.0325; visual cylinder length=0.025 radius=0.0325
- link base_link: mass 1.8 -> 0.5; geometry collision box size=0.18 0.10 0.003; visual box size=0.01 0.03 0.03
Joints:
- removed joint camera_joint
- removed joint joint_fl
- removed joint joint_fr
- removed joint joint_rl
- removed joint joint_rr
- added joint fl_steering_joint: type revolute, parent base_link, child fl_steering_knuckle, origin xyz=0.07 0.06 0.0 rpy=0 0 0, axis 0 0 1, limit lower=-0.78 upper=0.78 effort=5.0 velocity=10.0
- added joint fl_wheel_joint: type continuous, parent fl_steering_knuckle, child fl_wheel, origin xyz=0 0.02 0 rpy=0 0 0, axis 0 1 0
- added joint fr_steering_joint: type revolute, parent base_link, child fr_steering_knuckle, origin xyz=0.07 -0.06 0.0 rpy=0 0 0, axis 0 0 1, limit lower=-0.78 upper=0.78 effort=5.0 velocity=10.0
- added joint fr_wheel_joint: type continuous, parent fr_steering_knuckle, child fr_wheel, origin xyz=0 -0.02 0 rpy=0 0 0, axis 0 1 0
- added joint rl_wheel_joint: type continuous, parent base_link, child rl_wheel, origin xyz=-0.07 0.08 0 rpy=0 0 0, axis 0 1 0, limit effort=1.0 velocity=20.0
- added joint rr_wheel_joint: type continuous, parent base_link, child rr_wheel, origin xyz=-0.07 -0.08 0 rpy=0 0 0, axis 0 1 0, limit effort=1.0 velocity=20.0
